File: breadboardDuino.kicad_pcb (KiCad board)
At the start: 2 copper layers, 15 parts, among them J3 D-OUT, J4 A-OUT, J5 P-OUT, SW1 SPST, U1 ATMEGA328-PU, X1 16MHZ

Commit message: Inital layout
Parts:
- added J6: D-OUT2, conn-100mil:CONN-100MIL-M-1x5, F.Cu at (160.0, 108.0)
- J3: value D-OUT -> D-OUT1; footprint conn-100mil:CONN-100MIL-F-1x14 -> conn-100mil:CONN-100MIL-M-1x9
- moved R1 57.8 mm to (129.5, 132.1)
- moved JP2 52.1 mm to (125.7, 114.3)
- moved C3 48.4 mm to (124.5, 127.0), turned to 90 degrees
- moved SW1 42.8 mm to (129.5, 127.0), turned to 90 degrees
- moved C1 29.0 mm to (143.5, 125.7)
- moved J5 25.2 mm to (167.6, 127.0), turned to 180 degrees
- moved X1 21.1 mm to (149.9, 125.7), turned to 0 degrees
- moved C2 20.7 mm to (156.2, 125.7)
- moved C4 20.1 mm to (167.6, 130.8), turned to 0 degrees
- moved LED1 14.0 mm to (170.2, 109.2), turned to 90 degrees
- moved JP1 13.7 mm to (171.4, 116.8), turned to 270 degrees
- moved R2 12.0 mm to (174.0, 109.2), turned to 90 degrees
- moved J3 5.08 mm to (148.6, 130.8)
Connections:
- U1 pad 15: Net-(J3-Pad10) -> Net-(J6-Pad1)
- U1 pad 16: Net-(J3-Pad11) -> Net-(J6-Pad2)
Routing:
- net VCC: track 60.1 -> 108.2 mm, vias 0 -> 2
- net GND: track 74.3 -> 111.0 mm, vias 0 -> 1
- net /RESET: track 31.4 -> 62.0 mm, vias 0 -> 1
- net Net-(C1-Pad2): track 0.00 -> 22.5 mm
- net /RX: track 6.13 -> 25.3 mm
- net /TX: track 6.13 -> 22.7 mm
- net Net-(J3-Pad6): track 0.00 -> 15.3 mm
- net Net-(J3-Pad9): track 0.00 -> 12.8 mm
- net Net-(C2-Pad2): track 0.00 -> 12.5 mm
- net /MISO: track 31.0 -> 19.1 mm
- net /SCK: track 41.5 -> 32.8 mm
- net Net-(J3-Pad4): track 6.13 -> 13.5 mm
- net /MOSI: track 29.2 -> 21.9 mm
- net Net-(J3-Pad3): track 6.13 -> 12.8 mm
- net Net-(J3-Pad5): track 6.13 -> 11.7 mm
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
Commit message: Added some proto on the eges
Parts:
- added J1: CONN-100MIL-M-1x10, conn-100mil:CONN-100MIL-M-1x10, F.Cu at (179.1, 119.4)
- added J2: CONN-100MIL-M-1x10, conn-100mil:CONN-100MIL-M-1x10, F.Cu at (182.9, 119.4)
- added J7: CONN-100MIL-M-1x10, conn-100mil:CONN-100MIL-M-1x10, F.Cu at (120.7, 119.4)
- renumbered SW1 to ?
Routing:
- net VCC: track 108.2 -> 132.4 mm
- net GND: track 111.0 -> 126.5 mm
Other:
- board outline added: 67.3 x 27.9 mm

Commit message: Finished layout
Parts:
- removed ?: SPST, switches:B3F-10XX
- added SW1: SPST, switches:B3F-10XX, F.Cu at (130.8, 127.0)
- moved J1 58.4 mm to (120.7, 119.4)
- moved J7 54.6 mm to (175.3, 119.4)
- moved C4 43.2 mm to (124.5, 130.8), turned to 90 degrees
- moved J5 26.1 mm to (149.9, 108.0), turned to 0 degrees
- moved JP1 11.7 mm to (168.9, 128.3)
- moved R2 9.16 mm to (168.9, 116.8)
- moved J2 2.54 mm to (180.3, 119.4)
- moved C3 1.80 mm to (125.7, 125.7)
Connections:
- J1 pad 8: Net-(J1-Pad8) -> /RX
- J1 pad 9: Net-(J1-Pad9) -> /TX
Routing:
- net VCC: track 132.4 -> 107.5 mm, vias 2 -> 0
- net GND: track 126.5 -> 148.0 mm, vias 1 -> 2
- net /SCK: track 32.8 -> 47.4 mm, vias 0 -> 1
- net /MOSI: track 21.9 -> 33.3 mm
- net /TX: track 22.7 -> 29.9 mm
- net /RX: track 25.3 -> 32.5 mm
- net /MISO: track 19.1 -> 25.0 mm
- net /DTR: track 5.61 -> 3.81 mm
- net Net-(LED1-Pad1): track 5.39 -> 4.34 mm
- net /RESET: track 62.0 -> 61.3 mm, vias 1 -> 2
- added copper zone on B.Cu, net GND
Other:
- board size 67.3 x 27.9 mm -> 64.8 x 27.9 mm
- board text added: "A0"
- board text added: "A5"
- board text added: "D0"
- board text added: "D13"
- board text added: "D8"
- board text added: "D9"
- board text added: "FTDI"
- board text added: "GND"
- board text added: "ISP"
- board text added: "RX"
- board text added: "TX"
- board text added: "VCC"
- board text added: "myDuino v0.1"
